File: hardware/bypass.kicad_sch (KiCad schematic)
At the start: 6 parts, among them K1 G6K-2, K2 G6K-2, Q1 SS8050

Commit message: Reset references and remove THT footprint assignments.
Parts:
- renumbered R65 to R71
Changed lines of the file:
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@@
 		(on_board yes)
 		(dnp no)
-		(property "Reference" "R65"
+		(property "Reference" "R71"
 			(at 99.06 104.14 90)
 			(effects
@@
 			(project "Zero-Stomp"
 				(path "/8c8d5801-9c58-4283-98ac-c6a8e7250e15/5979a6af-2ef4-4435-a66c-af668b515c08"
-					(reference "R65")
+					(reference "R71")
 					(unit 1)
 				)

Commit message: Footprint assignments
Parts:
- K1, K2: footprint (none) -> Relay_SMD:Relay_DPDT_Omron_G6K-2F-Y
- R71: footprint (none) -> Resistor_SMD:R_0603_1608Metric
Changed lines of the file:
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@@
 			)
 		)
-		(property "Footprint" ""
+		(property "Footprint" "Resistor_SMD:R_0603_1608Metric"
 			(at 99.06 110.998 90)
 			(effects
@@
 			)
 		)
-		(property "Footprint" ""
+		(property "Footprint" "Relay_SMD:Relay_DPDT_Omron_G6K-2F-Y"
 			(at 134.62 80.01 0)
 			(effects
@@
 			)
 		)
-		(property "Footprint" ""
+		(property "Footprint" "Relay_SMD:Relay_DPDT_Omron_G6K-2F-Y"
 			(at 134.62 132.08 0)
 			(effects
