File: hardware/preamp.kicad_sch (KiCad schematic)
At the start: 62 parts, among them U10 TLV9064, U11 TLV9061xDBV, U12 TLV9064

Commit message: Reset references and remove THT footprint assignments.
Parts:
- C41, C42, C43, C44, C52, C53, C54, C55, C56, C57, C58, C59: footprint Capacitor_THT:C_Rect_L4.0mm_W2.5mm_P2.50mm -> (none)
- C47, C48, C49, C50, C51, C62, C63, C64, C65: footprint Capacitor_THT:CP_Radial_D5.0mm_P2.00mm -> (none)
- L2, L3, L4, L5: footprint Inductor_THT:L_Axial_L6.6mm_D2.7mm_P2.54mm_Vertical_Vishay_IM-2 -> (none)
- R44: renamed from R38; footprint Resistor_THT:R_Axial_DIN0207_L6.3mm_D2.5mm_P2.54mm_Vertical -> (none)
- R45: renamed from R39; footprint Resistor_THT:R_Axial_DIN0207_L6.3mm_D2.5mm_P2.54mm_Vertical -> (none)
- R46: renamed from R40; footprint Resistor_THT:R_Axial_DIN0207_L6.3mm_D2.5mm_P2.54mm_Vertical -> (none)
- R47: renamed from R41; footprint Resistor_THT:R_Axial_DIN0207_L6.3mm_D2.5mm_P2.54mm_Vertical -> (none)
- R48: renamed from R42; footprint Resistor_THT:R_Axial_DIN0207_L6.3mm_D2.5mm_P2.54mm_Vertical -> (none)
- R49: renamed from R43; footprint Resistor_THT:R_Axial_DIN0207_L6.3mm_D2.5mm_P2.54mm_Vertical -> (none)
- R50: renamed from R44; footprint Resistor_THT:R_Axial_DIN0207_L6.3mm_D2.5mm_P2.54mm_Vertical -> (none)
- R51: renamed from R45; footprint Resistor_THT:R_Axial_DIN0207_L6.3mm_D2.5mm_P2.54mm_Vertical -> (none)
- R52: renamed from R46; footprint Resistor_THT:R_Axial_DIN0207_L6.3mm_D2.5mm_P2.54mm_Vertical -> (none)
- R53: renamed from R47; footprint Resistor_THT:R_Axial_DIN0207_L6.3mm_D2.5mm_P2.54mm_Vertical -> (none)
- R54: renamed from R48; footprint Resistor_THT:R_Axial_DIN0207_L6.3mm_D2.5mm_P2.54mm_Vertical -> (none)
- R55: renamed from R49; footprint Resistor_THT:R_Axial_DIN0207_L6.3mm_D2.5mm_P2.54mm_Vertical -> (none)
- R60: renamed from R54; footprint Resistor_THT:R_Axial_DIN0207_L6.3mm_D2.5mm_P2.54mm_Vertical -> (none)
- R61: renamed from R55; footprint Resistor_THT:R_Axial_DIN0207_L6.3mm_D2.5mm_P2.54mm_Vertical -> (none)
- R62: renamed from R56; footprint Resistor_THT:R_Axial_DIN0207_L6.3mm_D2.5mm_P2.54mm_Vertical -> (none)
- R63: renamed from R57; footprint Resistor_THT:R_Axial_DIN0207_L6.3mm_D2.5mm_P2.54mm_Vertical -> (none)
- renumbered R32 to R38, R33 to R39, R34 to R40, R35 to R41, R36 to R42, R37 to R43, R50 to R56, R51 to R57, R52 to R58, R53 to R59

Commit message: Footprint assignments
Parts:
- removed C46, C61, C66, C67, C68, C69: 0u1, symbol Device:C_Polarized
- added C46, C61, C66, C67, C68, C69: 0u1, Capacitor_SMD:C_0603_1608Metric, symbol Device:C
- C41, C42, C43, C44, C52, C53, C54, C55: footprint (none) -> Capacitor_SMD:C_0603_1608Metric
- C45, C60: footprint (none) -> Capacitor_SMD:CP_Elec_4x5.4
- C47: footprint (none) -> Capacitor_Tantalum_SMD:CP_EIA-3528-21_Kemet-B
- C48, C49, C50, C51: value 1u -> 10u; footprint (none) -> Capacitor_Tantalum_SMD:CP_EIA-3216-18_Kemet-A
- C56, C57, C58, C59: footprint (none) -> Capacitor_SMD:C_0805_2012Metric
- C62, C63, C64, C65: footprint (none) -> Capacitor_Tantalum_SMD:CP_EIA-3216-18_Kemet-A
- L2, L3, L4, L5: footprint (none) -> Inductor_SMD:L_1210_3225Metric
- R38, R39, R40, R41, R42, R43, R48, R49, R50, R51, R56, R57, R58, R59: footprint (none) -> Resistor_SMD:R_0805_2012Metric
- R44, R45, R46, R47, R52, R53, R54, R55, R60, R61, R62, R63: footprint (none) -> Resistor_SMD:R_0603_1608Metric
- U10, U12: footprint (none) -> Package_SO:TSSOP-14_4.4x5mm_P0.65mm
Connections:
- net +5V_ISO: now also C46.1, C61.1
- net GNDA: now also C46.2, C61.2, C66.2, C67.2, C68.2, C69.2
- net at C65.2, L5.2, R63.1: now also C69.1
- net at C63.2, L3.2, R61.1: now also C67.1
- net at C62.2, L2.2, R60.1: now also C66.1
- net at C64.2, L4.2, R62.1: now also C68.1
