File: hardware/codec.kicad_sch (KiCad schematic)
At the start: 30 parts, among them J15 AudioJack4, U7 AP2112K-3.3, U8 AP2112K-1.8, U9 TLV320AIC3104

Commit message: Reset references and remove THT footprint assignments.
Parts:
- R30: renamed from R24; footprint Resistor_SMD:R_0805_2012Metric_Pad1.20x1.40mm_HandSolder -> (none)
- R31: renamed from R25; footprint Resistor_SMD:R_0805_2012Metric_Pad1.20x1.40mm_HandSolder -> (none)
- R32: renamed from R26; footprint Resistor_SMD:R_0805_2012Metric_Pad1.20x1.40mm_HandSolder -> (none)
- R33: renamed from R27; footprint Resistor_SMD:R_0805_2012Metric_Pad1.20x1.40mm_HandSolder -> (none)
- R34: renamed from R28; footprint Resistor_SMD:R_0805_2012Metric_Pad1.20x1.40mm_HandSolder -> (none)
- R35: renamed from R29; footprint Resistor_SMD:R_0805_2012Metric_Pad1.20x1.40mm_HandSolder -> (none)
- R36: renamed from R30; footprint Resistor_SMD:R_0805_2012Metric_Pad1.20x1.40mm_HandSolder -> (none)
- renumbered R31 to R37, TP6 to TP5, TP7 to TP6
Changed lines of the file:
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@@
 		(on_board yes)
 		(dnp no)
-		(property "Reference" "R26"
+		(property "Reference" "R32"
 			(at 106.426 83.82 90)
 			(effects
@@
 			)
 		)
-		(property "Footprint" "Resistor_SMD:R_0805_2012Metric_Pad1.20x1.40mm_HandSolder"
+		(property "Footprint" ""
 			(at 111.76 86.868 90)
 			(effects
@@
 			(project "Zero-Stomp"
 				(path "/8c8d5801-9c58-4283-98ac-c6a8e7250e15/99222d0b-8c34-4910-99fb-15750ad3fd36"
-					(reference "R26")
+					(reference "R32")
 					(unit 1)
 				)
@@
 		(on_board yes)
 		(dnp no)
-		(property "Reference" "R30"
+		(property "Reference" "R36"
 			(at 106.426 93.98 90)
 			(effects
@@
 			)
 		)
-		(property "Footprint" "Resistor_SMD:R_0805_2012Metric_Pad1.20x1.40mm_HandSolder"
+		(property "Footprint" ""
 			(at 111.76 97.028 90)
 			(effects
@@
 			(project "Zero-Stomp"
 				(path "/8c8d5801-9c58-4283-98ac-c6a8e7250e15/99222d0b-8c34-4910-99fb-15750ad3fd36"
-					(reference "R30")
+					(reference "R36")
 					(unit 1)
 				)
@@
 		(on_board yes)
 		(dnp no)
-		(property "Reference" "TP6"
+		(property "Reference" "TP5"
 			(at 100.33 85.09 90)
 			(effects
@@
 			(project ""
 				(path "/8c8d5801-9c58-4283-98ac-c6a8e7250e15/99222d0b-8c34-4910-99fb-15750ad3fd36"
-					(reference "TP6")
+					(reference "TP5")
 					(unit 1)
 				)
@@
 		(on_board yes)
 		(dnp no)
-		(property "Reference" "R25"
+		(property "Reference" "R31"
 			(at 106.934 71.374 0)
 			(effects
@@
 			)
 		)
-		(property "Footprint" "Resistor_SMD:R_0805_2012Metric_Pad1.20x1.40mm_HandSolder"
+		(property "Footprint" ""
 			(at 103.632 72.39 90)
 			(effects
@@
 			(project "Zero-Stomp"
 				(path "/8c8d5801-9c58-4283-98ac-c6a8e7250e15/99222d0b-8c34-4910-99fb-15750ad3fd36"
-					(reference "R25")
+					(reference "R31")
 					(unit 1)
 				)
@@
 		(on_board yes)
 		(dnp no)
-		(property "Reference" "R31"
+		(property "Reference" "R37"
 			(at 169.672 91.44 90)
 			(effects
@@
 			(project "Zero-Stomp"
 				(path "/8c8d5801-9c58-4283-98ac-c6a8e7250e15/99222d0b-8c34-4910-99fb-15750ad3fd36"
-					(reference "R31")
+					(reference "R37")
 					(unit 1)
 				)
@@
 		(on_board yes)
 		(dnp no)
-		(property "Reference" "R28"
+		(property "Reference" "R34"
 			(at 106.426 88.9 90)
 			(effects
@@
 			)
 		)
-		(property "Footprint" "Resistor_SMD:R_0805_2012Metric_Pad1.20x1.40mm_HandSolder"
+		(property "Footprint" ""
 			(at 111.76 91.948 90)
 			(effects
@@
 			(project "Zero-Stomp"
 				(path "/8c8d5801-9c58-4283-98ac-c6a8e7250e15/99222d0b-8c34-4910-99fb-15750ad3fd36"
-					(reference "R28")
+					(reference "R34")
 					(unit 1)
 				)
@@
 		(on_board yes)
 		(dnp no)
-		(property "Reference" "R24"
+		(property "Reference" "R30"
 			(at 99.06 71.1199 0)
 			(effects
@@
 			)
 		)
-		(property "Footprint" "Resistor_SMD:R_0805_2012Metric_Pad1.20x1.40mm_HandSolder"
+		(property "Footprint" ""
 			(at 103.378 72.39 90)
 			(effects
@@
 			(project "Zero-Stomp"
 				(path "/8c8d5801-9c58-4283-98ac-c6a8e7250e15/99222d0b-8c34-4910-99fb-15750ad3fd36"
-					(reference "R24")
+					(reference "R30")
 					(unit 1)
 				)
@@
 		(on_board yes)
 		(dnp no)
-		(property "Reference" "TP7"
+		(property "Reference" "TP6"
 			(at 114.3 100.33 90)
 			(effects
@@
 			(project "Zero-Stomp"
 				(path "/8c8d5801-9c58-4283-98ac-c6a8e7250e15/99222d0b-8c34-4910-99fb-15750ad3fd36"
-					(reference "TP7")
+					(reference "TP6")
 					(unit 1)
 				)
@@
 		(on_board yes)
 		(dnp no)
-		(property "Reference" "R27"
+		(property "Reference" "R33"
 			(at 106.426 86.36 90)
 			(effects
@@
 			)
 		)
-		(property "Footprint" "Resistor_SMD:R_0805_2012Metric_Pad1.20x1.40mm_HandSolder"
+		(property "Footprint" ""
 			(at 111.76 89.408 90)
 			(effects
@@
 			(project "Zero-Stomp"
 				(path "/8c8d5801-9c58-4283-98ac-c6a8e7250e15/99222d0b-8c34-4910-99fb-15750ad3fd36"
-					(reference "R27")
+					(reference "R33")
 					(unit 1)
 				)
@@
 		(on_board yes)
 		(dnp no)
-		(property "Reference" "R29"
+		(property "Reference" "R35"
 			(at 106.426 91.44 90)
 			(effects
@@
 			)
 		)
-		(property "Footprint" "Resistor_SMD:R_0805_2012Metric_Pad1.20x1.40mm_HandSolder"
+		(property "Footprint" ""
 			(at 111.76 94.488 90)
 			(effects
@@
 			(project "Zero-Stomp"
 				(path "/8c8d5801-9c58-4283-98ac-c6a8e7250e15/99222d0b-8c34-4910-99fb-15750ad3fd36"
-					(reference "R29")
-					(unit 1)
-				)
+					(reference "R35")
+					(unit 1)
+				)

Commit message: Footprint assignments
Parts:
- removed C29, C31, C34, C38, C40: 0u1, symbol Device:C_Polarized
- removed C35: 0.1u, symbol Device:C_Polarized_Small
- added C29, C31, C34, C38, C40: 0u1, Capacitor_SMD:C_0603_1608Metric, symbol Device:C
- added C35: 0u1, Capacitor_SMD:C_0603_1608Metric, symbol Device:C_Small
- C25, C26, C27, C28: footprint (none) -> Capacitor_SMD:C_0603_1608Metric
- C30, C32, C33, C37, C39: footprint (none) -> Capacitor_SMD:CP_Elec_4x5.4
- C36: footprint (none) -> Capacitor_SMD:CP_Elec_5x5.4
- J15: footprint (none) -> Connector_JST:JST_PH_B4B-PH-K_1x04_P2.00mm_Vertical
- R30, R31, R32, R33, R34, R35, R36, R37: footprint (none) -> Resistor_SMD:R_0603_1608Metric
- TP5: footprint (none) -> TestPoint:TestPoint_Pad_D1.0mm
- TP6: footprint TestPoint:TestPoint_Pad_D1.5mm -> TestPoint:TestPoint_Pad_D1.0mm
Connections:
- net +1V8: now also C31.1
- net +3V3: now also C29.1
- net GND: now also C29.2, C31.2
- net GNDA: now also C34.2, C38.2, C40.2
- net VDDA: now also C34.1, C38.1, C40.1
- net at J15.R2, R37.2, U9.14 (MIC2L/LINE2L/MICDET): now also C35.2
- net at U9.16 (MIC2R/LINE2R): now also C35.1

Commit message: Change connectors to JST SH
Parts:
- J15: value AudioJack4 -> HEADPHONE; footprint Connector_JST:JST_PH_B4B-PH-K_1x04_P2.00mm_Vertical -> Connector_JST:JST_PH_S4B-PH-K_1x04_P2.00mm_Horizontal
Changed lines of the file:
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@@
 			)
 		)
-		(property "Value" "AudioJack4"
+		(property "Value" "HEADPHONE"
 			(at 196.85 76.8351 0)
 			(effects
@@
 			)
 		)
-		(property "Footprint" "Connector_JST:JST_PH_B4B-PH-K_1x04_P2.00mm_Vertical"
+		(property "Footprint" "Connector_JST:JST_PH_S4B-PH-K_1x04_P2.00mm_Horizontal"
 			(at 187.96 80.01 0)
 			(effects
